Commit message: 20190401

File: schunk/urdf/pg70.urdf.xacro (robot description, xacro)
@@ -1,4 +1,4 @@
 <?xml version="1.0"?>
-<robot xmlns:xacro="http://www.ros.org/wiki/xacro">
+<robot name="chuanci" xmlns:xacro="http://www.ros.org/wiki/xacro">
   <xacro:include filename="$(find schunk)/urdf/common.xacro" />
   <xacro:include filename="$(find schunk)/urdf/pg70.gazebo.xacro" />
@@ -18,10 +18,14 @@
       <visual>
         <geometry>
-          <mesh filename="package://schunk/meshes/pg70.dae" />
+          <mesh filename="package://schunk/meshes/pg70_plus.stl "  />
+          <!--mesh filename="package://schunk/meshes/pg70_plus.stl " scale="0.001 0.001 0.001"/>
+          <mesh filename="package://schunk/meshes/pg70.dae" /-->
         </geometry>
       </visual>
       <collision>
         <geometry>
-          <mesh filename="package://schunk/meshes/pg70.stl" />
+          <mesh filename="package://schunk/meshes/pg70_plus.stl "  />
+          <!--mesh filename="package://schunk/meshes/pg70_plus.stl " scale="0.001 0.001 0.001" />
+          <mesh filename="package://schunk/meshes/pg70.stl" /-->
         </geometry>
       </collision>
